File: mbedTNC.brd (EAGLE design)
At the start: 66.7 x 32.9 mm, 61 parts, among them J1 SS-7066-NF, Q1 8Mhz, Q2 MMBT2222A, U1 MKL25ZXXVLH4, U10 MAX2674EWT+T, U2 S25FL208K0RMFI013, U3 MCP4661-XXXX_ML, U5 BMP180, U6 LMV358, U7 MCP73831, U8 TPS61201, X1 SMA003.062, X2 MICRO-USB-ZX62R-B-5P

Commit message: Version 1
Parts:
- removed C22: 22uF, SparkFun-Capacitors:1206
- removed SWD: SWD-10_SMD, mbed-HDK:SWD-10-SMD
- removed U10: MAX2674EWT+T, wrea:21-0217D_W61B1-1
- added C15: UWX1C100MCL2GB, wrea:PCAP_4X5.4-ELECT
- added R13: 33, SparkFun-Resistors:0603-RES
- added R14: 82, SparkFun-Resistors:0603-RES
- added R15: 1K, SparkFun-Resistors:0603-RES
- added R7: 10k, SparkFun-Resistors:0603-RES
- added U$4: VLP-ZZZ-X, wrea:VLP-ZZZ-X
- added U4: BMP280, wrea:BMP280
- added U9: TPS61201, texas:S-PDSO-N10
- C1: value 100pF -> 1.0uF
- C10: value 22pF -> 10uF; device SparkFun-Capacitors:0603-CAP -> SparkFun-Capacitors:0805
- C11: value 22pF -> 100pF
- C12: value 0.1uF -> 10pF
- C13: value 0.1uF -> 39pF
- C14: value UWX1C100MCL2GB -> 100pF; device wrea:PCAP_4X5.4-ELECT -> SparkFun-Capacitors:0603-CAP
- C16: device SparkFun-Capacitors:0603-CAP -> SparkFun:0603-CAP
- C17: value 0.1uF -> 4.7uF; device SparkFun-Capacitors:0603-CAP -> SparkFun-Capacitors:0805
- C19: value 4.7uF -> 10uF
- C2: value 10pF -> 1.0uF
- C20: value 10uF -> 1uF; device SparkFun-Capacitors:0805 -> SparkFun-Capacitors:0603-CAP
- C21: value 1uF -> 22uF; device SparkFun-Capacitors:0603-CAP -> SparkFun-Capacitors:1206
- C3: value 39pF -> 1.0uF
- C4: value 100pF -> 0.1uF
- C5: value 0.1uF -> 22pF; device SparkFun:0603-CAP -> SparkFun-Capacitors:0603-CAP
- C6: value 1.0uF -> 22pF
- C7, C8: value 1.0uF -> 0.1uF
- C9: value 0.1uF -> 10uF; device SparkFun-Capacitors:0603-CAP -> SparkFun-Capacitors:0805
- Q1: device wibauxl:CRYSTAL_5X3.2 -> wrea:CRYSTAL_5X3.2
- R1: value 25.5k -> 1M
- R10: value 33 -> 15
- R11: value 82 -> 5.6
- R12: value 1K -> 33
- R2: value 15 -> 2.2k; device SparkFun-Resistors:0603-RES -> SparkFun-Passives:0603-RES
- R3: value 5.6 -> 2.2k; device SparkFun-Resistors:0603-RES -> SparkFun-Passives:0603-RES
- R4: value 1M -> 1K
- R5, R6: value 2.2k -> 10k; device SparkFun-Passives:0603-RES -> SparkFun-Resistors:0603-RES
- R8: value 1K -> 10k
- R9: value 33 -> 25.5k
- U$1: value AF816M157502-T -> JTI_ANTENNA-1575AT43A40; device wrea:AF816 -> ava:JTI_ANTENNA-1575AT43A40
- U$2: value VLP-ZZZ-X -> SWD-10; device wrea:VLP-ZZZ-X -> wrea:M50-3600542
- U2: value S25FL208K0RMFI013 -> BMP180; device wrea:SO-8_SOA008 -> SparkFun-Sensors:BMP180
- U3: value MCP4661-XXXX_ML -> MAX2674EWT+T; device wrea:QFN16_4X4MC -> wrea:21-0217D_W61B1-1
- U5: value BMP180 -> LMV358; device SparkFun-Sensors:BMP180 -> wrea:DDU8-M
- U6: value LMV358 -> S25FL208K0RMFI013; device wrea:DDU8-M -> wrea:SO-8_SOA008
- U7: value MCP73831 -> MCP4661-XXXX_ML; device SparkFun:SOT23-5 -> wrea:QFN16_4X4MC
- U8: value TPS61201 -> MCP73831; device texas:S-PDSO-N10 -> SparkFun:SOT23-5
- moved R4 46.5 mm to (48.4, 30.6)
- moved C11 45.3 mm to (52.7, 2.35)
- moved C17 43.2 mm to (2.36, 26.6), turned to 180 degrees
- moved C1 40.8 mm to (11.9, 2.01)
- moved R11 39.7 mm to (41.9, 30.3)
- moved R9 39.2 mm to (48.5, 8.97)
- moved R1 39.1 mm to (9.61, 5.00), turned to 270 degrees
- moved C10 37.6 mm to (42.0, 24.5)
- moved C2 36.5 mm to (14.0, 2.01)
- moved C9 35.4 mm to (46.0, 24.5), turned to 0 degrees
- moved C3 33.7 mm to (16.1, 2.01), turned to 270 degrees
- moved R10 32.5 mm to (41.9, 28.2)
- moved R3 31.1 mm to (24.8, 5.33), turned to 180 degrees
- moved C4 30.4 mm to (18.1, 2.01)
- moved C12 29.8 mm to (50.5, 3.33)
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- renumbered JP5 to JP3
Connections:
- removed net N$12: C1.2, U$1.FEED
- removed net N$18: R10.1, X2.3
- new net D++: R13.1, X2.3
- new net D--: R12.1, X2.4
- net 3.3V: now also C1.1, C10.1, C2.1, C21.1, C3.1, C4.1, R10.2, R11.2, R6.1, R7.2, R8.1, U$2.P$1, U2.2, U2.3, U4.2, U4.6, U4.8, U5.8, U7.15, U9.10, U9.2; no longer C12.1, C13.1, C17.1, C22.1, C5.1, C6.1, R5.2, R6.2, SWD.P$1, U2.8, U3.15, U5.2, U5.3, U8.10, U8.2
- net AUDIO_IN: now also U5.1, U7.7; no longer U3.7, U6.1
- net AUDIO_OUT: now also C15.2; no longer C14.2
- net CARRIER_IN: now also U5.6, U5.7; no longer U6.6, U6.7
- net CRG_LED_AN: now also R14.1; no longer R11.1
- net CRG_LED_CATH: now also U8.1; no longer U7.1
- net D+: now also R13.2; no longer R10.2
- net D-: now also R12.2; no longer R9.2
- net DAC: now also U7.9; no longer U3.9
- net GND: now also C1.2, C10.2, C4.2, C5.1, C6.1, R15.2, R5.1, U$2.P$3, U$2.P$5, U$2.P$7, U$2.P$9, U2.7, U3.B2, U3.C1, U4.1, U4.5, U4.7, U5.4, U7.10, U7.13, U7.14, U7.17, U7.3, U7.4, U7.5, U8.2, U9.4, U9.9, U9.PP, U9.PP@1, U9.PP@2; no longer C10.1, C11.1, C22.2, C5.2, C6.2, R12.2, SWD.P$3, SWD.P$5, SWD.P$7, SWD.P$9, U10.B2, U10.C1, U2.4, U3.10, U3.13, U3.14, U3.17, U3.3, U3.4, U3.5, U5.7, U7.2, U8.4, U8.9, U8.PP, U8.PP@1, U8.PP@2
- net N$1: now also C11.2, U$1.FEED; no longer R9.1, X2.4
- net N$10: now also U9.3; no longer U8.3
- net N$11: now also C5.2, Q1.P$2, R1.1; no longer C10.2, Q1.2, R4.1
- net N$13: now also C6.2, Q1.P$1, R1.2; no longer C11.2, Q1.1, R4.2
- net N$15: now also R11.1; no longer R3.1
- net N$17: now also R10.1; no longer R2.1
- net N$19: now also C11.1; no longer C1.1
- net N$2: now also C14.1, R9.2, U3.A2; no longer C4.1, R1.2, U10.A2
- net N$21: now also C15.1, U7.8; no longer C14.1, U3.8
- net N$22: now also U5.3; no longer U6.3
- net N$24: now also R4.1; no longer R8.1
- net N$25: now also U5.5; no longer U6.5
- net N$26: now also U3.C2; no longer U10.C2
- net N$27: now also C13.1, R9.1; no longer C3.1, R1.1
- net N$4: now also U3.B1; no longer U10.B1
- net N$6: now also C17.1, R14.2, U8.4; no longer C18.1, R11.2, U7.4
- net N$7: now also C18.1, U8.3; no longer C19.1, U7.3
- net N$8: now also C12.1, U3.A1; no longer C2.1, U10.A1
- net N2: now also C14.2; no longer C4.2
- net NRESET: now also U$2.P$10; no longer SWD.P$10
- net P1W: now also U5.2, U7.6; no longer U3.6, U6.2
- net PROG1: now also R15.1, U8.5; no longer R12.1, U7.5
- net PTT: now also R4.2; no longer R8.2
- net RX_0: now also R7.1, U$2.P$8; no longer SWD.P$8
- net SCL: now also R2.1, U2.5, U4.4, U7.1; no longer R5.1, U3.1, U5.5
- net SDA: now also R3.1, U2.6, U4.3, U7.2; no longer R6.1, U3.2, U5.6
- net SPI0_MISO: now also U6.2; no longer U2.2
- net SPI0_MOSI: now also U6.5; no longer U2.5
- net SPI0_PCS0: now also U6.1; no longer U2.1
- net SPI0_SCK: now also U6.6; no longer U2.6
- net TCK: now also R5.2, U$2.P$4; no longer SWD.P$4
- net TMS: now also R6.2, U$2.P$2; no longer SWD.P$2
- net TX_0: now also R8.2, U$2.P$6; no longer SWD.P$6
- net VAUX: now also C20.1, U9.1; no longer C21.1, U8.1
- net VIN: now also C19.1, U9.5, U9.6, U9.7, U9.8; no longer C20.1, U8.5, U8.6, U8.7, U8.8
Routing:
- net 3.3V: track 63.6 -> 72.3 mm, vias 15 -> 19
- net D--: track 0.00 -> 7.19 mm
- net D++: track 0.00 -> 6.62 mm
- net N$18: track 6.31 -> 0.00 mm
- net TCK: track 29.5 -> 34.0 mm
- net GND: track 9.81 -> 5.48 mm, vias 151 -> 165
- net CRG_LED_AN: track 46.9 -> 50.9 mm
- net SCL: track 39.1 -> 43.1 mm, vias 2 -> 3
- net SDA: track 43.0 -> 46.5 mm
- net TX_LED: track 44.3 -> 41.1 mm
- net N$1: track 6.88 -> 3.76 mm
- net N$12: track 2.81 -> 0.00 mm
- net RX_0: track 30.5 -> 33.3 mm
- net N$24: track 7.26 -> 5.07 mm
- net GPS_LED: track 30.9 -> 28.7 mm
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Other:
- outline, holes or cut-outs redrawn
- board text added: "10"
- board text added: "V1"
