File: mbedTNC.sch (EAGLE design)
At the start: 58 parts, among them IC1 MKL25ZXXVLH4, IC2 TPS61201, IC3 LMV321-SOT-23-5, J1 MAX5481ETE, J2 SS-7066-NF, Q2 MMBT2222A, Q3 8Mhz, SW3 SPST_TACT-KMR2, U1 BMP180, U2 MCP73831, U3 MAX2659ELT+T, U4 S25FL208K0RMFI013

Commit message: Update
Added support for Yaesu/Icom radios. Moved components around.
Parts:
- removed IC3: LMV321-SOT-23-5, dp_devices:LMV321-SOT-23-5
- added JP2, JP4: JUMPER-PTH-2-NO, SparkFun-Passives:JUMPER-PTH-2-NO
- added R11: 1K, SparkFun-Resistors:RESISTOR0603
- added U$2: PVA2, wrea:PVA2
- added U5: LMV358, wrea:LMV358
- C5: value F921C105MPA -> 10uF; device wrea:F921C105MPA -> SparkFun-Capacitors:CAP0805; MPN F921C105MPA -> CL21A106KOQNNNE
- JP1: value USB-RECEPTABLE -> USB_MICROB_PLUGCONN-11752; device daspilker:USB-RECEPTABLE -> SparkFun-Connectors:USB_MICROB_PLUGCONN-11752
Connections:
- new net N$24: JP2.1, Q2.B, R11.1
- new net N$25: J2.5, U5B.+IN
- new net N$26: U$2.WIPER, U5A.-IN
- net 3.3V: now also U5B.V+; no longer IC3.V+
- net AUDIO_IN: now also U$2.CCW, U5A.OUT; no longer IC3.-, IC3.OUT
- net AUDIO_OUT: now also C5.2, JP4.2; no longer C5.-
- net CARRIER_IN: now also U5B.-IN, U5B.OUT; no longer J2.5
- net GND: now also Q2.E, U$2.CW, U5B.V-; no longer IC3.GND, Q2.C
- net N$21: now also C5.1; no longer C5.+
- net N$22: now also U5A.+IN; no longer IC3.+
- net N$3: now also Q2.C; no longer Q2.E
- net PTT: now also JP2.2, JP4.1, R11.2; no longer Q2.B
Other:
- moved on the sheet: JP1, Q2

Commit message: Update
Changed to a 2 circuit digipot. Various other changes
Parts:
- removed C22: 0.1uF, SparkFun-Capacitors:CAP0603-CAP
- removed J1: MAX5481ETE, wrea:MAX5481ETE
- removed JP4: JUMPER-PTH-2-NO, SparkFun-Passives:JUMPER-PTH-2-NO
- removed R8: 10k, SparkFun-Resistors:RESISTOR0603
- removed U$2: PVA2, wrea:PVA2
- added J3: 1981568-1, wrea:1981568-1
- added U6: MCP4661-XXXX_ML, wrea:MCP4661-XXXX_ML
- JP1: value USB_MICROB_PLUGCONN-11752 -> JUMPER-PTH-2-NO; device SparkFun-Connectors:USB_MICROB_PLUGCONN-11752 -> SparkFun-Passives:JUMPER-PTH-2-NO; MPN 10103594-0001LF -> (none)
- R6, R7: value 4.7K -> 2.2k; MPN RMCF0603FT4K70 -> RMCF0603JT2K20
Connections:
- removed net N$19: C22.1, J1.17, J1.GND, J1.VSS, J1.VSS_2
- removed net N$26: U$2.WIPER, U5A.-IN
- removed net SPI1_MISO: IC1.PTD7, U4.SO
- removed net SPI1_MOSI: IC1.PTD6, U4.SI/IO0
- removed net SPI1_PCS0: IC1.PTD4, U4.*CS
- removed net SPI1_SCK: IC1.PTD5, U4.SCK
- new net P1W: U5A.-IN, U6.P1W
- net 3.3V: now also U6.VDD; no longer J1.SPI/*UD, J1.VDD
- net AUDIO_IN: now also U6.P1A; no longer U$2.CCW
- net AUDIO_OUT: now also JP2.2; no longer JP4.2
- net CARRIER_IN: now also IC1.PTB1; no longer IC1.PTE21
- net DAC: now also U6.P0W; no longer J1.H
- net GND: now also J3.1, U6.A1, U6.A2, U6.EP, U6.P0B, U6.P1B, U6.VSS, U6.VSS_2; no longer C22.2, J1.L, JP1.GND, R8.2, U$2.CW
- net N$1: now also J3.4; no longer JP1.D-
- net N$18: now also J3.3; no longer JP1.D+
- net N$21: now also U6.P0A; no longer J1.W
- net N$24: now also JP1.1; no longer JP2.1
- net N$6: now also J3.5; no longer JP1.VCC
- net PTT: now also JP1.2, JP2.1; no longer JP2.2, JP4.1
- net SCL: now also R6.1, U6.SCL; no longer R7.1
- net SDA: now also R7.1, U6.SDA; no longer R6.1
- net SPI0_MISO: now also U4.SO; no longer IC1.PTD3, J1.DIN_U/*D
- net SPI0_MOSI: now also U4.SI/IO0
- net SPI0_PCS0: now also U4.*CS; no longer J1.*CS
- net SPI0_SCK: now also U4.SCK; no longer J1.SCLK_*INC
- net TMS: no longer R8.1
Other:
- moved on the sheet: C5, JP2, R6, R7, SWD

Commit message: Update.
Move to 4 layer board. New LNA with internal switch for an active
external ant. Finalizing parts, moved stuff around.
Parts:
- removed BAT1: (no value), SparkFun-Electromechanical:BATTERY12MM
- removed C15: 1.0uF, SparkFun-Capacitors:CAP0603-CAP
- removed IC1: MKL25ZXXVLH4, wrea:MKL25ZXXVLH4
- removed IC2: TPS61201, texas:TPS61201
- removed J3: 1981568-1, wrea:1981568-1
- removed JP3: LiPo Battery, SparkFun:M02-JST-2MM-SMT
- removed R13, R14: 33, SparkFun-Resistors:RESISTOR0603
- removed R7: 2.2k, SparkFun-Passives:RESISTOR0603-RES
- removed SW3: SPST_TACT-KMR2, adafruit:SPST_TACT-KMR2
- removed U$4: AF816M157502-T, wrea:AF816M157502-T
- removed U4: S25FL208K0RMFI013, wrea:S25FL208K0RMFI013
- added BATT1: BK-890, wrea:BK-890
- added C21: 1uF, SparkFun-Capacitors:CAP0603-CAP
- added C22: 22uF, SparkFun-Capacitors:CAP1206
- added JP4: LiPo Battery, SparkFun:M02-JST-2MM-SMT
- added JP5: PTH-JUMPER-3-NO, wrea:PTH-JUMPER-3-NO
- added R12, R8: 1K, SparkFun-Resistors:RESISTOR0603
- added RESET: JUMPER-PAD-2-NOYES_SILK, SparkFun-Passives:JUMPER-PAD-2-NOYES_SILK
- added U$2: VLP-ZZZ-X, wrea:VLP-ZZZ-X
- added U10: MAX2674EWT+T, wrea:MAX2674EWT+T
- added U7: MCP73831, SparkFun:MCP73831
- added U8: TPS61201, texas:TPS61201
- added X1: SMA003.062, wrea:SMA003.062
- added X2: MICRO-USB-ZX62R-B-5P, con-hirose:MICRO-USB-ZX62R-B-5P
- C1: value 0.1uF -> 100pF; device SparkFun:CAP0603-CAP -> SparkFun-Capacitors:CAP0603-CAP; MPN GRM188R71C104KA01D -> CL10B101KB8NNNC
- C10, C11: value 1.0uF -> 22pF; MPN GRM188R71C104KA01D -> C1608C0G1H220J080AA
- C14: value 0.1uF -> UWX1C100MCL2GB; device SparkFun-Capacitors:CAP0603-CAP -> wrea:UWX1C100MCL2GB; MPN GRM188R71C104KA01D -> UWX1C100MCL2GB
- C18, C19: value 22pF -> 4.7uF; device SparkFun-Capacitors:CAP0603-CAP -> SparkFun-Capacitors:CAP0805; MPN C1608C0G1H220J080AA -> CL21B475KOFNNNE
- C2: value 1.0uF -> 10pF; MPN GRM188R61C105KA93D -> CL10C100CB8NNNC
- C20: value 22uF -> 10uF; device SparkFun-Capacitors:CAP1206 -> SparkFun-Capacitors:CAP0805; MPN CL31A226KOCLFNC -> CL21A106KOQNNNE
- C3: value 0.1uF -> 39pF; MPN GRM188R71C104KA01D -> CL10C390JB8NNNC
- C4: value 10uF -> 100pF; device SparkFun-Capacitors:CAP0805 -> SparkFun-Capacitors:CAP0603-CAP; MPN CL21A106KOQNNNE -> CL10B101KB8NNNC
- C5: value 10uF -> 0.1uF; device SparkFun-Capacitors:CAP0805 -> SparkFun:CAP0603-CAP; MPN CL21A106KOQNNNE -> GRM188R71C104KA01D
- C6, C7: value 4.7uF -> 1.0uF; MPN EMK107ABJ475KA-T -> EMK107B7105KA-T
- C8: value 470pF -> 1.0uF; device SparkFun:CAP0402-CAP -> SparkFun-Capacitors:CAP0603-CAP; MPN VJ0603D471KXXAJ -> EMK107B7105KA-T
- C9: value 33nF -> 0.1uF; device SparkFun:CAP0402-CAP -> SparkFun-Capacitors:CAP0603-CAP; MPN (none) -> GRM188R71C104KA01D
- L1: value 4.7uH, 1.2A -> 91nH; device SparkFun-Passives:INDUCTOR. -> SparkFun-Passives:INDUCTOR0603; MPN CDRH2D18/HPNP-4R7NC -> LQW18AN91NJ00D
- L3: value 6.8nH -> BLM18HG102SN1D; device SparkFun:INDUCTOR0402 -> wrea:BLM18HG102SN1D; MPN ELJ-RE6N8ZFA -> BLM18HG102SN1D
- L4: value BLM18HG102SN1D -> 4.7uH, 1.2A; device wrea:BLM18HG102SN1D -> SparkFun-Passives:INDUCTOR.; MPN BLM18HG102SN1D -> CDRH2D18/HPNP-4R7NC
- R1: value 82 -> 25.5k; MPN ESR03EZPJ820 -> RMCF0603FT25K5
- R10: value 1M -> 33; MPN RMCF0603FT1M00 -> RMCF0603FT33R0
- R11: value 1K -> 82; MPN RMCF0603JT1K00 -> ESR03EZPJ820
- R2: value 1K -> 15; MPN RMCF0603JT1K00 -> RMCF0603JT15R0
- R3: value 10k -> 5.6; MPN RNCP0603FTD10K0 -> RMCF0603FT5R60
- R4: value 5.6 -> 1M; MPN RMCF0603FT5R60 -> RMCF0603FT1M00
- R5: value 10k -> 2.2k; device SparkFun-Resistors:RESISTOR0603 -> SparkFun-Passives:RESISTOR0603-RES; MPN RNCP0603FTD10K0 -> RMCF0603JT2K20
- R9: value 15 -> 33; MPN RMCF0603JT15R0 -> RMCF0603FT33R0
- S1: value (none) -> EG1270; device SparkFun-Electromechanical:SWITCH-SPDTSMD2 -> wrea:EG1270; MPN (none) -> EG1270
- SWD: MPN FTSH-105-01-F-D-K -> 20021321-00008C4LF
- U$1: value VLP-ZZZ-X -> AF816M157502-T; device wrea:VLP-ZZZ-X -> wrea:AF816M157502-T; MPN VLP-500-F -> AF816M157502-T
- U1: value BMP180 -> MKL25ZXXVLH4; device SparkFun-Sensors:BMP180 -> wrea:MKL25ZXXVLH4; MPN (none) -> MKL25ZXXVLH4
- U2: value MCP73831 -> S25FL208K0RMFI013; device SparkFun:MCP73831 -> wrea:S25FL208K0RMFI013; MPN MCP73831 -> S25FL208K0RMFI013
- U3: value MAX2659ELT+T -> MCP4661-XXXX_ML; device wrea:MAX2659ELT+T -> wrea:MCP4661-XXXX_ML; MPN (none) -> MCP6N11-010E/SN
- U5: value LMV358 -> BMP180; device wrea:LMV358 -> SparkFun-Sensors:BMP180; MPN PVA2A103A01R00 -> (none)
- U6: value MCP4661-XXXX_ML -> LMV358; device wrea:MCP4661-XXXX_ML -> wrea:LMV358; MPN (none) -> LMV358
- renumbered D3 to D1, J2 to J1, Q3 to Q1
Connections:
- removed net N$14: C9.2, U$3.14_VCC_RF, U3.VCC
- removed net N$9: C8.2, L3.1
- new net GPS_INT: U$3.5_EXTINT0, U1.PTD4
- new net N$19: C1.1, L1.1
- new net N$26: U10.ANT, X1.1
- new net N$27: C3.1, R1.1, U$3.13_ANTON
- new net N$28: BATT1.+, JP5.3
- new net N2: C4.2, U$3.11_RF_IN
- net 3.3V: now also C22.1, C5.1, C6.1, C7.1, C8.1, C9.1, JP5.1, R2.2, R3.2, U1.VDD1, U1.VDD2, U1.VDD3, U1.VDDA, U1.VREFH, U2.VCC, U3.VDD, U5.VDD, U5.VDDIO, U6B.V+, U8.FB, U8.VOUT; no longer C1.1, C10.1, C11.1, C14.1, C15.1, C20.1, IC1.VDD1, IC1.VDD2, IC1.VDD3, IC1.VDDA, IC1.VREFH, IC2.FB, IC2.VOUT, R4.2, R7.2, R9.2, U1.VDD, U1.VDDIO, U4.VCC, U5B.V+, U6.VDD
- net AUDIO_IN: now also U1.PTB0, U3.P1A, U6A.OUT; no longer IC1.PTB0, U5A.OUT, U6.P1A
- net AUDIO_OUT: now also C14.-; no longer C5.2
- net CARRIER_IN: now also U1.PTB1, U6B.-IN, U6B.OUT; no longer IC1.PTB1, U5B.-IN, U5B.OUT
- net CRG_LED_AN: now also R11.1; no longer R1.1
- net CRG_LED_CATH: now also U7.STAT; no longer U2.STAT
- net D+: now also R10.2, U1.USB_D+; no longer IC1.USB_D+, R13.2
- net D-: now also R9.2, U1.USB_D-; no longer IC1.USB_D-, R14.2
- net DAC: now also U1.PTE30, U3.P0W; no longer IC1.PTE30, U6.P0W
- net GND: now also BATT1.-, C10.1, C11.1, C18.2, C19.2, C21.2, C22.2, C5.2, C8.2, C9.2, JP4.1, R12.2, RESET.1, U1.VREFL, U1.VSS1, U1.VSS2, U1.VSS3, U1.VSSA, U10.GNDAC, U10.GNDDC, U2.GND, U3.A1, U3.A2, U3.EP, U3.P0B, U3.P1B, U3.VSS, U3.VSS_2, U5.GND, U6B.V-, U7.VSS, U8.GND, U8.PGND, U8.PP, U8.PP@1, U8.PP@2, X1.2, X2.1; no longer BAT1.-, C1.2, C10.2, C11.2, C14.2, C15.2, C18.1, C19.1, C4.2, C9.1, IC1.VREFL, IC1.VSS1, IC1.VSS2, IC1.VSS3, IC1.VSSA, IC2.GND, IC2.PGND, IC2.PP, IC2.PP@1, IC2.PP@2, J3.1, JP3.1, R2.2, R3.1, SW3.S, SW3.S1, U1.GND, U2.VSS, U3.GND, U3.GND_2, U4.GND, U5B.V-, U6.A1, U6.A2, U6.EP, U6.P0B, U6.P1B, U6.VSS, U6.VSS_2
- net N$1: now also R9.1, X2.4; no longer J3.4, R14.1
- net N$10: now also L4.1, U8.L; no longer IC2.L, L1.1
- net N$11: now also C10.2, R4.1, U1.XTALIN; no longer C18.2, IC1.XTALIN, R10.1
- net N$12: now also C1.2, U$1.FEED; no longer C8.1, U$4.FEED
- net N$13: now also C11.2, R4.2, U1.XTALOUT; no longer C19.2, IC1.XTALOUT, R10.2
- net N$15: now also R3.1; no longer R4.1
- net N$16: now also U1.PTC11; no longer IC1.PTC11
- net N$17: now also R2.1; no longer R9.1
- net N$18: now also R10.1, X2.3; no longer J3.3, R13.1
- net N$2: now also C4.1, R1.2, U10.RFOUT/*SHDN; no longer U$3.11_RF_IN, U3.RFOUT
- net N$21: now also C14.+, U3.P0A; no longer C5.1, U6.P0A
- net N$22: now also U6A.+IN; no longer U5A.+IN
- net N$23: now also L3.2; no longer L4.2
- net N$24: now also R8.1; no longer R11.1
- net N$25: now also U6B.+IN; no longer U5B.+IN
- net N$4: now also L1.2, U10.RFIN; no longer R3.2, U$3.13_ANTON, U3.*SHDN
- net N$5: now also JP5.2; no longer BAT1.+
- net N$6: now also C18.1, R11.2, U7.VIN, X2.5; no longer C6.1, J3.5, R1.2, U2.VIN
- net N$7: now also C19.1, JP4.2, U7.VBAT; no longer C7.1, JP3.2, U2.VBAT
- net N$8: now also C2.1, U$3.14_VCC_RF, U10.VCC; no longer L3.2, U3.RFIN
- net NRESET: now also RESET.2, U1.NRESET; no longer C2.1, IC1.NRESET, R5.1, SW3.P, SW3.P1
- net P1W: now also U3.P1W, U6A.-IN; no longer U5A.-IN, U6.P1W
- net PROG1: now also R12.1, U7.PROG; no longer R2.1, U2.PROG
- net PTT: now also R8.2, U1.PTE22; no longer IC1.PTE22, R11.2
- net RX_0: now also L3.1, U1.PTA1; no longer IC1.PTA1, L4.1
- net SCL: now also R5.1, U1.PTC1, U3.SCL, U5.SCL; no longer IC1.PTC1, R6.1, U1.SCL, U6.SCL
- net SDA: now also R6.1, U1.PTC2, U3.SDA, U5.SDA; no longer IC1.PTC2, R7.1, U1.SDA, U6.SDA
- net SPI0_MISO: now also U2.SO; no longer U4.SO
- net SPI0_MOSI: now also U1.PTD2, U2.SI/IO0; no longer IC1.PTD2, U4.SI/IO0
- net SPI0_PCS0: now also U1.PTD0, U2.*CS; no longer IC1.PTD0, U4.*CS
- net SPI0_SCK: now also U1.PTD1, U2.SCK; no longer IC1.PTD1, U4.SCK
- net TCK: now also U1.SWCLK; no longer IC1.SWCLK
- net TMS: now also U1.SWDIO; no longer IC1.SWDIO
- net TX_0: now also U1.PTA2; no longer IC1.PTA2
- net TX_LED: now also U1.PTC10; no longer IC1.PTC10
- net VAUX: now also C21.1, U8.VAUX; no longer C3.1, IC2.VAUX
- net VIN: now also C20.1, L4.2, S1.O2, U8.EN, U8.PS, U8.UVLO, U8.VIN; no longer C4.1, IC2.EN, IC2.PS, IC2.UVLO, IC2.VIN, L1.2, S1.S

Commit message: Version 1
Parts:
- removed C22: 22uF, SparkFun-Capacitors:CAP1206
- removed JP5: PTH-JUMPER-3-NO, wrea:PTH-JUMPER-3-NO
- removed SWD: SWD-10_SMD, mbed-HDK:SWD-10_SMD
- removed U10: MAX2674EWT+T, wrea:MAX2674EWT+T
- added C15: UWX1C100MCL2GB, wrea:UWX1C100MCL2GB
- added JP3: PTH-JUMPER-3-NO, wrea:PTH-JUMPER-3-NO
- added R13: 33, SparkFun-Resistors:RESISTOR0603
- added R14: 82, SparkFun-Resistors:RESISTOR0603
- added R15: 1K, SparkFun-Resistors:RESISTOR0603
- added R7: 10k, SparkFun-Resistors:RESISTOR0603
- added U$4: VLP-ZZZ-X, wrea:VLP-ZZZ-X
- added U4: BMP280, wrea:BMP280
- added U9: TPS61201, texas:TPS61201
- C1: value 100pF -> 1.0uF; MPN CL10B101KB8NNNC -> EMK107B7105KA-T
- C10: value 22pF -> 10uF; device SparkFun-Capacitors:CAP0603-CAP -> SparkFun-Capacitors:CAP0805; MPN C1608C0G1H220J080AA -> CC0805KKX5R6BB106
- C11: value 22pF -> 100pF; MPN C1608C0G1H220J080AA -> CL10B101KB8NNNC
- C12: value 0.1uF -> 10pF; MPN GRM188R71C104KA01D -> CL10C100CB8NNNC
- C13: value 0.1uF -> 39pF; MPN GRM188R71C104KA01D -> CL10C390JB8NNNC
- C14: value UWX1C100MCL2GB -> 100pF; device wrea:UWX1C100MCL2GB -> SparkFun-Capacitors:CAP0603-CAP; MPN UWX1C100MCL2GB -> CL10B101KB8NNNC
- C16: device SparkFun-Capacitors:CAP0603-CAP -> SparkFun:CAP0603-CAP
- C17: value 0.1uF -> 4.7uF; device SparkFun-Capacitors:CAP0603-CAP -> SparkFun-Capacitors:CAP0805; MPN GRM188R71C104KA01D -> CL21B475KOFNNNE
- C19: value 4.7uF -> 10uF; MPN CL21B475KOFNNNE -> CL21A106KOQNNNE
- C2: value 10pF -> 1.0uF; MPN CL10C100CB8NNNC -> EMK107B7105KA-T
- C20: value 10uF -> 1uF; device SparkFun-Capacitors:CAP0805 -> SparkFun-Capacitors:CAP0603-CAP; MPN CL21A106KOQNNNE -> EMK107B7105KA-T
- C21: value 1uF -> 22uF; device SparkFun-Capacitors:CAP0603-CAP -> SparkFun-Capacitors:CAP1206; MPN EMK107B7105KA-T -> CL31A226KOCLFNC
- C3: value 39pF -> 1.0uF; MPN CL10C390JB8NNNC -> EMK107B7105KA-T
- C4: value 100pF -> 0.1uF; MPN CL10B101KB8NNNC -> GRM188R71C104KA01D
- C5: value 0.1uF -> 22pF; device SparkFun:CAP0603-CAP -> SparkFun-Capacitors:CAP0603-CAP; MPN GRM188R71C104KA01D -> C1608C0G1H220J080AA
- C6: value 1.0uF -> 22pF; MPN EMK107B7105KA-T -> C1608C0G1H220J080AA
- C7, C8: value 1.0uF -> 0.1uF; MPN EMK107B7105KA-T -> GRM188R71C104KA01D
- C9: value 0.1uF -> 10uF; device SparkFun-Capacitors:CAP0603-CAP -> SparkFun-Capacitors:CAP0805; MPN GRM188R71C104KA01D -> CC0805KKX5R6BB106
- D1: MPN (none) -> LRTBGFTM-ST7-1+VV9-29+Q5R
- JP4: MPN (none) -> S2B-PH-SM4-TB(LF)(SN)
- Q1: device wibauxl:CRYSTAL_5X3.2 -> wrea:CRYSTALCRYSTAL_5X3.2
- R1: value 25.5k -> 1M; MPN RMCF0603FT25K5 -> RMCF0603FT1M00
- R10: value 33 -> 15; MPN RMCF0603FT33R0 -> RMCF0603JT15R0
- R11: value 82 -> 5.6; MPN ESR03EZPJ820 -> RMCF0603FT5R60
- R12: value 1K -> 33; MPN RMCF0603JT1K00 -> RMCF0603FT33R0
- R2: value 15 -> 2.2k; device SparkFun-Resistors:RESISTOR0603 -> SparkFun-Passives:RESISTOR0603-RES; MPN RMCF0603JT15R0 -> RMCF0603JT2K20
- R3: value 5.6 -> 2.2k; device SparkFun-Resistors:RESISTOR0603 -> SparkFun-Passives:RESISTOR0603-RES; MPN RMCF0603FT5R60 -> RMCF0603JT2K20
- R4: value 1M -> 1K; MPN RMCF0603FT1M00 -> RMCF0603JT1K00
- R5, R6: value 2.2k -> 10k; device SparkFun-Passives:RESISTOR0603-RES -> SparkFun-Resistors:RESISTOR0603; MPN RMCF0603JT2K20 -> RNCP0603FTD10K0
- R8: value 1K -> 10k; MPN RMCF0603JT1K00 -> RNCP0603FTD10K0
- R9: value 33 -> 25.5k; MPN RMCF0603FT33R0 -> RMCF0603FT25K5
- U$1: value AF816M157502-T -> JTI_ANTENNA-1575AT43A40; device wrea:AF816M157502-T -> ava:JTI_ANTENNA-1575AT43A40; MPN AF816M157502-T -> 1575AT43A0040E
- U$2: value VLP-ZZZ-X -> SWD-10; device wrea:VLP-ZZZ-X -> wrea:SWD-10; MPN VLP-500-F -> (none)
- U2: value S25FL208K0RMFI013 -> BMP180; device wrea:S25FL208K0RMFI013 -> SparkFun-Sensors:BMP180; MPN S25FL208K0RMFI013 -> (none)
- U3: value MCP4661-XXXX_ML -> MAX2674EWT+T; device wrea:MCP4661-XXXX_ML -> wrea:MAX2674EWT+T; MPN MCP6N11-010E/SN -> MAX2674EWT+T
- U5: value BMP180 -> LMV358; device SparkFun-Sensors:BMP180 -> wrea:LMV358; MPN (none) -> LMV358IDDUR
- U6: value LMV358 -> S25FL208K0RMFI013; device wrea:LMV358 -> wrea:S25FL208K0RMFI013; MPN LMV358 -> S25FL208K0RMFI013
- U7: value MCP73831 -> MCP4661-XXXX_ML; device SparkFun:MCP73831 -> wrea:MCP4661-XXXX_ML; MPN MCP73831 -> MCP4661T-103E/ML
- U8: value TPS61201 -> MCP73831; device texas:TPS61201 -> SparkFun:MCP73831; MPN (none) -> MCP73831
Connections:
- removed net N$12: C1.2, U$1.FEED
- removed net N$18: R10.1, X2.3
- new net D++: R13.1, X2.3
- new net D--: R12.1, X2.4
- net 3.3V: now also C1.1, C10.1, C2.1, C21.1, C3.1, C4.1, JP3.1, R10.2, R11.2, R6.1, R7.2, R8.1, U$2.1, U2.VDD, U2.VDDIO, U4.VDD, U4.VDDIO, U5B.V+, U6.VCC, U7.VDD, U9.FB, U9.VOUT; no longer C12.1, C13.1, C17.1, C22.1, C5.1, C6.1, JP5.1, R5.2, R6.2, SWD.P$1, U2.VCC, U3.VDD, U5.VDD, U5.VDDIO, U6B.V+, U8.FB, U8.VOUT
- net AUDIO_IN: now also U5A.OUT, U7.P1A; no longer U3.P1A, U6A.OUT
- net AUDIO_OUT: now also C15.-; no longer C14.-
- net CARRIER_IN: now also U5B.-IN, U5B.OUT; no longer U6B.-IN, U6B.OUT
- net CRG_LED_AN: now also R14.1; no longer R11.1
- net CRG_LED_CATH: now also U8.STAT; no longer U7.STAT
- net D+: now also R13.2; no longer R10.2
- net D-: now also R12.2; no longer R9.2
- net DAC: now also U7.P0W; no longer U3.P0W
- net GND: now also C1.2, C10.2, C4.2, C5.1, C6.1, R15.2, R5.1, U$2.3, U$2.5, U$2.7, U$2.9, U3.GNDAC, U3.GNDDC, U4.GND, U4.SDO, U5B.V-, U6.GND, U7.A1, U7.A2, U7.EP, U7.P0B, U7.P1B, U7.VSS_2, U8.VSS, U9.GND, U9.PGND, U9.PP, U9.PP@1, U9.PP@2; no longer C10.1, C11.1, C22.2, C5.2, C6.2, R12.2, SWD.P$3, SWD.P$5, SWD.P$7, SWD.P$9, U10.GNDAC, U10.GNDDC, U3.A1, U3.A2, U3.EP, U3.P0B, U3.P1B, U3.VSS, U3.VSS_2, U5.GND, U6B.V-, U8.GND, U8.PGND, U8.PP, U8.PP@1, U8.PP@2
- net N$1: now also C11.2, U$1.FEED; no longer R9.1, X2.4
- net N$10: now also U9.L; no longer U8.L
- net N$11: now also C5.2, R1.1; no longer C10.2, R4.1
- net N$13: now also C6.2, R1.2; no longer C11.2, R4.2
- net N$15: now also R11.1; no longer R3.1
- net N$17: now also R10.1; no longer R2.1
- net N$19: now also C11.1; no longer C1.1
- net N$2: now also C14.1, R9.2, U3.RFOUT/*SHDN; no longer C4.1, R1.2, U10.RFOUT/*SHDN
- net N$21: now also C15.+, U7.P0A; no longer C14.+, U3.P0A
- net N$22: now also U5A.+IN; no longer U6A.+IN
- net N$24: now also R4.1; no longer R8.1
- net N$25: now also U5B.+IN; no longer U6B.+IN
- net N$26: now also U3.ANT; no longer U10.ANT
- net N$27: now also C13.1, R9.1; no longer C3.1, R1.1
- net N$28: now also JP3.3; no longer JP5.3
- net N$4: now also U3.RFIN; no longer U10.RFIN
- net N$5: now also JP3.2; no longer JP5.2
- net N$6: now also C17.1, R14.2, U8.VIN; no longer C18.1, R11.2, U7.VIN
- net N$7: now also C18.1, U8.VBAT; no longer C19.1, U7.VBAT
- net N$8: now also C12.1, U3.VCC; no longer C2.1, U10.VCC
- net N2: now also C14.2; no longer C4.2
- net NRESET: now also U$2.10; no longer SWD.P$10
- net P1W: now also U5A.-IN, U7.P1W; no longer U3.P1W, U6A.-IN
- net PROG1: now also R15.1, U8.PROG; no longer R12.1, U7.PROG
- net PTT: now also R4.2; no longer R8.2
- net RX_0: now also R7.1, U$2.8; no longer SWD.P$8
- net SCL: now also R2.1, U2.SCL, U4.SCL, U7.SCL; no longer R5.1, U3.SCL, U5.SCL
- net SDA: now also R3.1, U2.SDA, U4.SDA, U7.SDA; no longer R6.1, U3.SDA, U5.SDA
- net SPI0_MISO: now also U6.SO; no longer U2.SO
- net SPI0_MOSI: now also U6.SI/IO0; no longer U2.SI/IO0
- net SPI0_PCS0: now also U6.*CS; no longer U2.*CS
- net SPI0_SCK: now also U6.SCK; no longer U2.SCK
- net TCK: now also R5.2, U$2.4; no longer SWD.P$4
- net TMS: now also R6.2, U$2.2; no longer SWD.P$2
- net TX_0: now also R8.2, U$2.6; no longer SWD.P$6
- net VAUX: now also C20.1, U9.VAUX; no longer C21.1, U8.VAUX
- net VIN: now also C19.1, U9.EN, U9.PS, U9.UVLO, U9.VIN; no longer C20.1, U8.EN, U8.PS, U8.UVLO, U8.VIN
Other:
- moved on the sheet: BATT1, C1, C10, C11, C12, C13, C16, C18, C19, C2, C20, C21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
